File: Circuits/SoftTakeover/SoftTakeover.sch (KiCad schematic (older format))
At the start: 13 parts, among them J1 Conn_01x08_Male, J2 Conn_01x08_Male, J3 Conn_ARM_JTAG_SWD_10, U1 ATSAMD11D14A-M, U2 MCP4728, U3 ADG734

Commit message: Added various schematics
Parts:
- removed R1: 10k, Resistor_SMD:R_0603_1608Metric, symbol Device:R
- added C5: 0.1uF, Capacitor_SMD:C_0603_1608Metric, symbol Device:C
- added C6: 1uF, Capacitor_SMD:C_0603_1608Metric, symbol Device:C
- C1, C2, C3, C4: value 100nF -> 0.1uF
Connections:
- net GND: now also C2.1, J3.9 (GNDDetect), C5.2, C6.2; no longer C2.2
- net RST: no longer C2.1
- net VDD: now also C2.2, C5.1, C6.1
- no-connect marks 11 -> 10
Other:
- moved on the sheet: C1
Changed lines of the file:
@@
 L power:VDD #PWR0102
 U 1 1 5FAD4A02
-P 2050 3250
-F 0 "#PWR0102" H 2050 3100 50  0001 C CNN
-F 1 "VDD" H 2065 3423 50  0000 C CNN
-F 2 "" H 2050 3250 50  0001 C CNN
-F 3 "" H 2050 3250 50  0001 C CNN
-	1    2050 3250
+P 2200 3150
+F 0 "#PWR0102" H 2200 3000 50  0001 C CNN
+F 1 "VDD" H 2215 3323 50  0000 C CNN
+F 2 "" H 2200 3150 50  0001 C CNN
+F 3 "" H 2200 3150 50  0001 C CNN
+	1    2200 3150
 	1    0    0    -1
 $EndComp
@@
 P 4200 3600
 F 0 "C4" H 4085 3554 50  0000 R CNN
-F 1 "100nF" H 4085 3645 50  0000 R CNN
+F 1 "0.1uF" H 4085 3645 50  0000 R CNN
 F 2 "Capacitor_SMD:C_0603_1608Metric" H 4238 3450 50  0001 C CNN
 F 3 "~" H 4200 3600 50  0001 C CNN
@@
 Wire Wire Line
 	3800 4450 3900 4450
-Text GLabel 1950 5950 2    50   Input ~ 0
-RST
-$Comp
-L Device:R R1
-U 1 1 5FAF7E6A
-P 1650 5800
-F 0 "R1" H 1720 5846 50  0000 L CNN
-F 1 "10k" H 1720 5755 50  0000 L CNN
-F 2 "Resistor_SMD:R_0603_1608Metric" V 1580 5800 50  0001 C CNN
-F 3 "~" H 1650 5800 50  0001 C CNN
-	1    1650 5800
-	1    0    0    -1
-$EndComp
-Wire Wire Line
-	1950 5950 1650 5950
-$Comp
-L Device:C C2
-U 1 1 5FAF8D8B
-P 1650 6100
-F 0 "C2" H 1765 6146 50  0000 L CNN
-F 1 "100nF" H 1765 6055 50  0000 L CNN
-F 2 "Capacitor_SMD:C_0603_1608Metric" H 1688 5950 50  0001 C CNN
-F 3 "~" H 1650 6100 50  0001 C CNN
-	1    1650 6100
-	1    0    0    -1
-$EndComp
-Connection ~ 1650 5950
-$Comp
-L power:VDD #PWR0105
-U 1 1 5FAFB065
-P 1650 5650
-F 0 "#PWR0105" H 1650 5500 50  0001 C CNN
-F 1 "VDD" H 1665 5823 50  0000 C CNN
-F 2 "" H 1650 5650 50  0001 C CNN
-F 3 "" H 1650 5650 50  0001 C CNN
-	1    1650 5650
-	1    0    0    -1
-$EndComp
-$Comp
-L power:GND #PWR0106
-U 1 1 5FAF9760
-P 1650 6250
-F 0 "#PWR0106" H 1650 6000 50  0001 C CNN
-F 1 "GND" H 1655 6077 50  0000 C CNN
-F 2 "" H 1650 6250 50  0001 C CNN
-F 3 "" H 1650 6250 50  0001 C CNN
-	1    1650 6250
-	1    0    0    -1
-$EndComp
-Wire Wire Line
-	1800 3250 2050 3250
+Wire Wire Line
+	1950 3150 2200 3150
 Text GLabel 5050 5250 2    50   Input ~ 0
 SDA_DAC
@@
 P 8500 4150
 F 0 "C3" H 8700 4150 50  0000 R CNN
-F 1 "100nF" H 8750 4250 50  0000 R CNN
+F 1 "0.1uF" H 8750 4250 50  0000 R CNN
 F 2 "Capacitor_SMD:C_0603_1608Metric" H 8538 4000 50  0001 C CNN
 F 3 "~" H 8500 4150 50  0001 C CNN
@@
 Wire Wire Line
 	7950 4650 8100 4650
-$Comp
-L Device:R R3
-U 1 1 5FB47E94
-P 7500 4600
-F 0 "R3" H 7570 4646 50  0000 L CNN
-F 1 "5k" H 7570 4555 50  0000 L CNN
-F 2 "Resistor_SMD:R_0603_1608Metric" V 7430 4600 50  0001 C CNN
-F 3 "~" H 7500 4600 50  0001 C CNN
-	1    7500 4600
-	1    0    0    -1
-$EndComp
 Wire Wire Line
 	7800 4650 7950 4650
@@
 L power:VDD #PWR0113
 U 1 1 5FB3F7CF
-P 9900 1600
-F 0 "#PWR0113" H 9900 1450 50  0001 C CNN
-F 1 "VDD" H 9915 1773 50  0000 C CNN
-F 2 "" H 9900 1600 50  0001 C CNN
-F 3 "" H 9900 1600 50  0001 C CNN
-	1    9900 1600
+P 9450 1600
+F 0 "#PWR0113" H 9450 1450 50  0001 C CNN
+F 1 "VDD" H 9465 1773 50  0000 C CNN
+F 2 "" H 9450 1600 50  0001 C CNN
+F 3 "" H 9450 1600 50  0001 C CNN
+	1    9450 1600
 	1    0    0    -1
 $EndComp
@@
 L Device:C C1
 U 1 1 5FC12197
-P 2050 3400
-F 0 "C1" H 2250 3400 50  0000 R CNN
-F 1 "100nF" H 2300 3500 50  0000 R CNN
-F 2 "Capacitor_SMD:C_0603_1608Metric" H 2088 3250 50  0001 C CNN
-F 3 "~" H 2050 3400 50  0001 C CNN
-	1    2050 3400
+P 2100 3400
+F 0 "C1" H 2300 3400 50  0000 R CNN
+F 1 "0.1uF" H 2350 3500 50  0000 R CNN
+F 2 "Capacitor_SMD:C_0603_1608Metric" H 2138 3250 50  0001 C CNN
+F 3 "~" H 2100 3400 50  0001 C CNN
+	1    2100 3400
 	-1   0    0    1
 $EndComp
@@
 L power:GND #PWR0114
 U 1 1 5FC128B1
-P 2050 3550
-F 0 "#PWR0114" H 2050 3300 50  0001 C CNN
-F 1 "GND" H 2055 3377 50  0000 C CNN
-F 2 "" H 2050 3550 50  0001 C CNN
-F 3 "" H 2050 3550 50  0001 C CNN
-	1    2050 3550
-	1    0    0    -1
-$EndComp
-Text GLabel 1800 3250 0    50   Input ~ 0
+P 2200 3550
+F 0 "#PWR0114" H 2200 3300 50  0001 C CNN
+F 1 "GND" H 2205 3377 50  0000 C CNN
+F 2 "" H 2200 3550 50  0001 C CNN
+F 3 "" H 2200 3550 50  0001 C CNN
+	1    2200 3550
+	1    0    0    -1
+$EndComp
+Text GLabel 1950 3150 0    50   Input ~ 0
 3v3
 Text GLabel 1600 1300 2    50   Input ~ 0
@@
 Text GLabel 1600 1700 2    50   Input ~ 0
 IN_3
-Connection ~ 2050 3250
 Text GLabel 6400 2100 1    50   Input ~ 0
 IN_1
@@
 NoConn ~ 4650 1900
 $Comp
-L power:GND #PWR?
+L power:GND #PWR0105
 U 1 1 5FE6A4A1
-P 4150 2300
-F 0 "#PWR?" H 4150 2050 50  0001 C CNN
-F 1 "GND" H 4155 2127 50  0000 C CNN
-F 2 "" H 4150 2300 50  0001 C CNN
-F 3 "" H 4150 2300 50  0001 C CNN
-	1    4150 2300
+P 4100 2300
+F 0 "#PWR0105" H 4100 2050 50  0001 C CNN
+F 1 "GND" H 4105 2127 50  0000 C CNN
+F 2 "" H 4100 2300 50  0001 C CNN
+F 3 "" H 4100 2300 50  0001 C CNN
+	1    4100 2300
 	1    0    0    -1
 $EndComp
@@
 $EndComp
 $Comp
-L power:VDD #PWR?
+L power:VDD #PWR0106
 U 1 1 5FE73FCC
 P 4150 1100
-F 0 "#PWR?" H 4150 950 50  0001 C CNN
+F 0 "#PWR0106" H 4150 950 50  0001 C CNN
 F 1 "VDD" H 4165 1273 50  0000 C CNN
 F 2 "" H 4150 1100 50  0001 C CNN
@@
 	1    0    0    -1
 $EndComp
-NoConn ~ 4050 2300
+Wire Wire Line
+	4050 2300 4100 2300
+Connection ~ 4100 2300
+Wire Wire Line
+	4100 2300 4150 2300
+Wire Wire Line
+	9900 1600 9450 1600
+$Comp
+L Device:C C5
+U 1 1 5FB7F2F7
+P 9450 1750
+F 0 "C5" H 9565 1796 50  0000 L CNN
+F 1 "0.1uF" H 9565 1705 50  0000 L CNN
+F 2 "Capacitor_SMD:C_0603_1608Metric" H 9488 1600 50  0001 C CNN
+F 3 "~" H 9450 1750 50  0001 C CNN
+	1    9450 1750
+	1    0    0    -1
+$EndComp
+Connection ~ 9450 1600
+$Comp
+L power:GND #PWR0116
+U 1 1 5FB82B72
+P 9450 1900
+F 0 "#PWR0116" H 9450 1650 50  0001 C CNN
+F 1 "GND" H 9455 1727 50  0000 C CNN
+F 2 "" H 9450 1900 50  0001 C CNN
+F 3 "" H 9450 1900 50  0001 C CNN
+	1    9450 1900
+	1    0    0    -1
+$EndComp
+$Comp
+L Device:C C6
+U 1 1 5FB831FA
+P 9200 1750
+F 0 "C6" H 8950 1750 50  0000 L CNN
+F 1 "1uF" H 8900 1650 50  0000 L CNN
+F 2 "Capacitor_SMD:C_0603_1608Metric" H 9238 1600 50  0001 C CNN
+F 3 "~" H 9200 1750 50  0001 C CNN
+	1    9200 1750
+	1    0    0    -1
+$EndComp
+Wire Wire Line
+	9200 1600 9450 1600
+Wire Wire Line
+	9200 1900 9450 1900
+Connection ~ 9450 1900
+$Comp
+L Device:C C2
+U 1 1 5FBB0CC4
+P 2300 3400
+F 0 "C2" H 2150 3400 50  0000 R CNN
+F 1 "0.1uF" H 2250 3500 50  0000 R CNN
+F 2 "Capacitor_SMD:C_0603_1608Metric" H 2338 3250 50  0001 C CNN
+F 3 "~" H 2300 3400 50  0001 C CNN
+	1    2300 3400
+	-1   0    0    1
+$EndComp
+Wire Wire Line
+	2100 3550 2200 3550
+Connection ~ 2200 3550
+Wire Wire Line
+	2200 3550 2300 3550
+Wire Wire Line
+	2100 3250 2200 3250
+Wire Wire Line
+	2200 3250 2200 3150
+Connection ~ 2200 3250
+Wire Wire Line
+	2200 3250 2300 3250
+Connection ~ 2200 3150
+$Comp
+L Device:R R3
+U 1 1 5FB47E94
+P 7500 4600
+F 0 "R3" H 7570 4646 50  0000 L CNN
+F 1 "5k" H 7570 4555 50  0000 L CNN
+F 2 "Resistor_SMD:R_0603_1608Metric" V 7430 4600 50  0001 C CNN
+F 3 "~" H 7500 4600 50  0001 C CNN
+	1    7500 4600
+	1    0    0    -1
+$EndComp
 $EndSCHEMATC
