File: Circuits/SoftTakeover/SoftTakeoverV1.kicad_pcb (KiCad board)
At the start: 2 copper layers, 31.8 x 21.6 mm, 13 parts, among them J1 Conn_01x08_Male, J2 Conn_01x08_Male, J3 Conn_ARM_JTAG_SWD_10, U1 ATSAMD11D14A-M, U2 MCP4728, U3 ADG734

Commit message: Added various schematics
Parts:
- removed J3: Conn_ARM_JTAG_SWD_10, Connector_PinHeader_1.27mm:PinHeader_2x05_P1.27mm_Vertical
- U1: value ATSAMD11D14A-M -> SAMD11D14AM
Connections:
- J2 pad 1: GND -> SWDIO
- J2 pad 2: 3v3 -> SWCLK
- J2 pad 8: Net-(J2-Pad8) -> RST
Routing:
- net GND: track 3.89 -> 46.5 mm, vias 1 -> 3
- net RST: track 41.1 -> 23.5 mm
- net SWCLK: track 16.4 -> 9.47 mm
- net SWDIO: track 13.9 -> 11.7 mm
- net 3v3: track 50.8 -> 49.0 mm
