File: Circuits/SoftTakeover/SoftTakeoverV2.kicad_pcb (KiCad board)
At the start: 2 copper layers, 31.8 x 21.6 mm, 12 parts, among them J1 Conn_01x08_Male, J2 Conn_01x08_Male, U1 SAMD11D14AM, U2 MCP4728, U3 ADG734

Commit message: Added various schematics
Parts:
- added J3: Conn_ARM_JTAG_SWD_10, Connector_PinHeader_1.27mm:PinHeader_2x05_P1.27mm_Vertical, F.Cu at (110.5, 95.2)
- U1: value SAMD11D14AM -> ATSAMD11D14A-M
Connections:
- J2 pad 1: SWDIO -> GND
- J2 pad 2: SWCLK -> 3v3
- J2 pad 8: RST -> Net-(J2-Pad8)
Routing:
- net 3v3: track 49.0 -> 68.5 mm
- net RST: track 23.5 -> 41.1 mm
- net GND: track 46.5 -> 32.2 mm, vias 3 -> 9
- net SWCLK: track 9.47 -> 16.4 mm
- net LAYER_SEL: track 15.6 -> 11.7 mm, vias 1 -> 3
- net SWDIO: track 11.7 -> 13.9 mm
- added copper zone on B.Cu, net GND
- added copper zone on F.Cu, net GND
Other:
- board text added: "Rev. 2"
